Commit message: did alot of testing with urdf, i think i got one model working, need to test in gazebo

File: ros2_ws/src/robot_visual/urdf/robot_visual.urdf.xacro (robot description, xacro)
@@ -1,92 +1,164 @@
-<?xml version="1.0" encoding="UTF-8"?>
-<!DOCTYPE xml>
-<robot xmlns:xacro="http://www.ros.org/wiki/xacro" name="robot_visual">
-  <xacro:property name="L1" value="0.20" />
-  <xacro:property name="L1radius" value="0.05" />
-  <xacro:property name="L2" value="0.15" />
-  <xacro:property name="L2radius" value="0.03" />
-  <xacro:property name="L3" value="0.08" />
-  <xacro:property name="L3radius" value="0.02" />
-  <xacro:property name="eesize" value="0.05" />
-  <xacro:property name="J1MIN" value="${-pi/2}" />
-  <xacro:property name="J1MAX" value="${pi/2}" />
-  <xacro:property name="J2MIN" value="-0.08" />
-  <xacro:property name="J2MAX" value="0.08" />
-  <xacro:property name="J3MIN" value="${-pi}" />
-  <xacro:property name="J3MAX" value="${pi}" />
-  <material name="blue">
-    <color rgba="0.2 0.4 0.65 1" />
-  </material>
-  <material name="yellow">
-    <color rgba="1 0.85 0 1" />
-  </material>
-  <link name="world" />
-  <link name="base" />
-  <link name="link1">
-    <visual name="link1">
-      <origin xyz="0 0 ${-L1/2}" />
-      <geometry>
-        <cylinder radius="${L1radius}" length="${L1}" />
-      </geometry>
-      <material name="blue" />
-    </visual>
-  </link>
-  <link name="link2">
-    <visual name="link2">
-      <origin xyz="0 0 0" />
-      <geometry>
-        <cylinder radius="${L2radius}" length="${2*L2}" />
-      </geometry>
-      <material name="blue" />
-    </visual>
-  </link>
-  <link name="link3">
-    <visual name="link3">
-      <origin xyz="0 0 ${L3/2}" />
-      <geometry>
-        <cylinder radius="${L3radius}" length="${L3}" />
-      </geometry>
-      <material name="blue" />
-    </visual>
-  </link>
-  <link name="ee">
-    <visual name="ee">
-      <origin xyz="0 0 0" />
-      <geometry>
-        <box size="${eesize} ${eesize} ${eesize}" />
-      </geometry>
-      <material name="yellow" />
-    </visual>
-  </link>
-  <joint name="base_in_world" type="fixed">
-    <parent link="world" />
-    <child link="base" />
-    <origin xyz="${-(L2+L3)} 0 0" rpy="0 0 ${pi/2}" />
-  </joint>
-  <joint name="joint1" type="revolute">
-    <parent link="base" />
-    <child link="link1" />
-    <origin xyz="0 0 ${L1}" rpy="0 0 0" />
-    <axis xyz="0 0 1" />
-    <limit lower="${J1MIN}" upper="${J1MAX}" effort="1" velocity="1" />
-  </joint>
-  <joint name="joint2" type="prismatic">
-    <parent link="link1" />
-    <child link="link2" />
-    <origin xyz="0 0 0" rpy="${pi/2} 0 0" />
-    <axis xyz="0 0 1" />
-    <limit lower="${J2MIN}" upper="${J2MAX}" effort="1" velocity="1" />
-  </joint>
-  <joint name="joint3" type="revolute">
-    <parent link="link2" />
-    <child link="link3" />
-    <origin xyz="0 0 ${L2}" rpy="0 0 0" />
-    <axis xyz="0 0 1" />
-    <limit lower="${J3MIN}" upper="${J3MAX}" effort="1" velocity="1" />
-  </joint>
-  <joint name="ee_in_link3" type="fixed">
-    <parent link="link3" />
-    <child link="ee" />
-    <origin xyz="0 0 ${L3}" rpy="0 0 0" />
-  </joint>
+<?xml version="1.0"?>
+<robot xmlns:xacro="http://www.ros.org/wiki/xacro">
+    <xacro:include filename="inertial_macros.xacro"/>
+    <xacro:property name="track_radius" value="0.04"/>
+    <xacro:property name="track_length" value="0.27"/>
+    <xacro:property name="track_width" value="0.04"/>
+    <material name="white">
+        <color rgba="1 1 1 1" />
+    </material>
+    <material name="orange">
+        <color rgba="1 0.3 0.1 1"/>
+    </material>
+    <material name="blue">
+        <color rgba="0.2 0.2 1 1"/>
+    </material>
+    <material name="black">
+        <color rgba="0 0 0 1"/>
+    </material>
+    <!-- BASE LINK -->
+    <link name="base_link">
+    </link>
+    <!-- CHASSIS LINK -->
+    <joint name="chassis_joint" type="fixed">
+        <parent link="base_link"/>
+        <child link="chassis"/>
+        <origin xyz="0 0 0"/>
+    </joint>
+    <link name="chassis">
+        <visual>
+            <origin xyz="0 0 0.075"/>
+            <geometry>
+                <box size="0.3 0.3 0.15"/>
+            </geometry>
+            <material name="white"/>
+        </visual>
+        <collision>
+            <origin xyz="0 0 0.075"/>
+            <geometry>
+                <box size="0.3 0.3 0.15"/>
+            </geometry>
+        </collision>
+        <xacro:inertial_box mass="0.5" x="0.3" y="0.3" z="0.15">
+            <origin xyz="0 0 0.075" rpy="0 0 0"/>
+        </xacro:inertial_box>
+    </link>
+    <gazebo reference="chassis">
+        <material>Gazebo/White</material>
+    </gazebo>
+    <!-- LEFT WHEEL LINK -->
+    <joint name="left_wheel_joint" type="continuous">
+        <parent link="base_link"/>
+        <child link="left_wheel"/>
+        <origin xyz="0 0.2 0" rpy="0 0 0" />
+    </joint>
+    <link name="left_wheel">
+        <visual>
+            <geometry>
+                <box size="${2*track_radius - track_length} ${track_width} ${track_radius*2} "/>
+            </geometry>
+            <material name="blue"/>
+        </visual>
+        <collision>
+            <geometry>
+                <box size="${2*track_radius - track_length} ${track_width} ${track_radius*2} "/>
+            </geometry>
+        </collision>
+        <xacro:inertial_box mass="0.1" x="${2*track_radius - track_length}" y="${track_width}" z="${track_radius*2}" >
+            <origin xyz="0 0 0" rpy="0 0 0"/>
+        </xacro:inertial_box>
+        <visual>
+            <origin xyz="${track_length/2 + - track_radius} 0.0 0.0" rpy="${pi/2} 0.0 0.0"/>
+            <geometry>
+                <cylinder radius="${track_radius}" length="${track_width}"/>
+            </geometry>
+            <material name="blue"/>
+        </visual>
+        <collision>
+            <origin xyz="${track_length/2 + - track_radius} 0.0 0.0" rpy="${pi/2} 0.0 0.0"/>
+            <geometry>
+                <cylinder radius="${track_radius}" length="${track_width}"/>
+            </geometry>
+        </collision>
+        <xacro:inertial_cylinder mass="0.05" length="${track_radius}" radius="${track_width}">
+            <origin xyz="${track_length/2 + - track_radius} 0.0 0.0" rpy="${pi/2} 0.0 0.0"/>
+        </xacro:inertial_cylinder>
+        <visual>
+            <origin xyz="${-track_length/2 + track_radius} 0.0 0.0" rpy="${pi/2} 0.0 0.0"/>
+            <geometry>
+                <cylinder radius="${track_radius}" length="${track_width}"/>
+            </geometry>
+            <material name="blue"/>
+        </visual>
+        <collision>
+            <origin xyz="${-track_length/2 + track_radius} 0.0 0.0" rpy="${pi/2} 0.0 0.0"/>
+            <geometry>
+                <cylinder radius="${track_radius}" length="${track_width}"/>
+            </geometry>
+        </collision>
+        <xacro:inertial_cylinder mass="0.05" length="${track_radius}" radius="${track_width}">
+            <origin xyz="${-track_length/2 + track_radius} 0.0 0.0" rpy="${pi/2} 0.0 0.0"/>
+        </xacro:inertial_cylinder>
+    </link>
+    <gazebo reference="left_wheel">
+        <material>Gazebo/Blue</material>
+    </gazebo>
+    <!-- RIGHT WHEEL LINK -->
+    <joint name="right_wheel_joint" type="continuous">
+        <parent link="base_link"/>
+        <child link="right_wheel"/>
+        <origin xyz="0 -0.2 0" rpy="0 0 0" />
+    </joint>
+    <link name="right_wheel">
+        <visual>
+            <geometry>
+                <box size="${2*track_radius - track_length} ${track_width} ${track_radius*2} "/>
+            </geometry>
+            <material name="blue"/>
+        </visual>
+        <collision>
+            <geometry>
+                <box size="${2*track_radius - track_length} ${track_width} ${track_radius*2} "/>
+            </geometry>
+        </collision>
+        <xacro:inertial_box mass="0.1" x="${2*track_radius - track_length}" y="${track_width}" z="${track_radius*2}" >
+            <origin xyz="0 0 0" rpy="0 0 0"/>
+        </xacro:inertial_box>
+        <visual>
+            <origin xyz="${track_length/2 + - track_radius} 0.0 0.0" rpy="${pi/2} 0.0 0.0"/>
+            <geometry>
+                <cylinder radius="${track_radius}" length="${track_width}"/>
+            </geometry>
+            <material name="blue"/>
+        </visual>
+        <collision>
+            <origin xyz="${track_length/2 + - track_radius} 0.0 0.0" rpy="${pi/2} 0.0 0.0"/>
+            <geometry>
+                <cylinder radius="${track_radius}" length="${track_width}"/>
+            </geometry>
+        </collision>
+        <xacro:inertial_cylinder mass="0.05" length="${track_radius}" radius="${track_width}">
+            <origin xyz="${track_length/2 + - track_radius} 0.0 0.0" rpy="${pi/2} 0.0 0.0"/>
+        </xacro:inertial_cylinder>
+        <visual>
+            <origin xyz="${-track_length/2 + track_radius} 0.0 0.0" rpy="${pi/2} 0.0 0.0"/>
+            <geometry>
+                <cylinder radius="${track_radius}" length="${track_width}"/>
+            </geometry>
+            <material name="blue"/>
+        </visual>
+        <collision>
+            <origin xyz="${-track_length/2 + track_radius} 0.0 0.0" rpy="${pi/2} 0.0 0.0"/>
+            <geometry>
+                <cylinder radius="${track_radius}" length="${track_width}"/>
+            </geometry>
+        </collision>
+        <xacro:inertial_cylinder mass="0.05" length="${track_radius}" radius="${track_width}">
+            <origin xyz="${-track_length/2 + track_radius} 0.0 0.0" rpy="${pi/2} 0.0 0.0"/>
+        </xacro:inertial_cylinder>
+    </link>
+    <gazebo
+        reference="right_wheel">
+        <material>Gazebo/Blue</material>
+    </gazebo>
 </robot>
