Commit message: trying something

File: ros2_ws/src/thesis_robot/urdf/robot_visual.urdf.xacro (robot description, xacro)
@@ -10,10 +10,10 @@
     <xacro:property name="wheel_thickness" value="0.041"/>
     <xacro:property name="wheel_mass" value="0.05"/>
-    <xacro:property name="wheel_offset_x" value="0.02"/>
+    <xacro:property name="wheel_offset_x" value="0.24"/>
     <xacro:property name="wheel_offset_y" value="0.1"/>
     <xacro:property name="wheel_offset_z" value="0.01"/>
     <xacro:property name="caster_wheel_radius" value="0.01"/>
     <xacro:property name="caster_wheel_mass" value="0.01"/>
-    <xacro:property name="caster_wheel_offset_x" value="0.24"/>
+    <xacro:property name="caster_wheel_offset_x" value="0.02"/>
     <xacro:property name="caster_wheel_offset_z" value="${wheel_offset_z - wheel_radius + caster_wheel_radius}"/>
     <material name="white">
