Commit message: fixed tf i think

File: ros2_ws/src/thesis_robot/urdf/lidar.xacro (robot description, xacro)
@@ -4,5 +4,5 @@
         <parent link="chassis"/>
         <child link="laser"/>
-        <origin xyz="0.21 0 0.175" rpy="0 0 0"/>
+        <origin xyz="0.1 0 0.175" rpy="0 0 ${pi}"/>
     </joint>
     <link name="laser">
